Commit message: fixed launch file

File: smartcar_simulation/urdf/sensors.xacro (robot description, xacro)
@@ -5,5 +5,5 @@
     <link name="imu_link">
         <visual>
-            <origin xyz="${wheelbase_length / 2} 0 ${wheel_diameter}" rpy="0 0 0"/>
+            <origin xyz="0 0 ${wheel_diameter}" rpy="0 0 0"/>
             <geometry>
                 <box size="${imu_size} ${imu_size} ${imu_size}"/>
