Commit message: added sensors, gazebo & driving

File: smartcar_simulation/urdf/materials.xacro (robot description, xacro)
@@ -1,4 +1,7 @@
 <?xml version="1.0"?>
 <robot xmlns:xacro="http://www.ros.org/wiki/xacro">
+    <material name="body_material">
+        <color rgba="1 0 0 1"/>
+    </material>
     <material name="wheel_material">
         <color rgba="0 0 0 1"/>
@@ -8,5 +11,5 @@
     </material>
     <material name="lidar_material">
-        <color rgba="0 0 0 1"/>
+        <color rgba="1 0 1 1"/>
     </material>
     <material name="footprint_material">

File: smartcar_simulation/urdf/sensors.xacro (robot description, xacro)
@@ -5,5 +5,5 @@
     <link name="imu_link">
         <visual>
-            <origin xyz="0 0 ${wheel_diameter}" rpy="0 0 0"/>
+            <origin xyz="0 0 0" rpy="0 0 0"/>
             <geometry>
                 <box size="${imu_size} ${imu_size} ${imu_size}"/>
@@ -11,4 +11,17 @@
             <material name="imu_material"/>
         </visual>
+        <collision>
+            <origin xyz="0 0 0" rpy="0 0 0"/>
+            <geometry>
+                <box size="${imu_size} ${imu_size} ${imu_size}"/>
+            </geometry>
+        </collision>
+        <inertial>
+            <mass value="0.1"/>
+            <origin xyz="0 0 0" rpy="0 0 0"/>
+            <inertia ixx="0.00001" ixy="0.0" ixz="0.0" iyy="0.00001" iyz="0.0" izz="0.00001"/>
+        </inertial>
+    </link>
+    <gazebo reference="imu_link">
         <sensor name="my_imu" type="imu">
             <always_on>true</always_on>
@@ -16,12 +29,12 @@
             <plugin name="my_imu_plugin" filename="libgazebo_ros_imu_sensor.so">
                 <ros>
-                <!-- Will publish to /imu_data -->
-                <namespace></namespace>
-                <remapping>~/out:=imu_data</remapping>
+                    <remapping>~/out:=imu_data</remapping>
                 </ros>
             </plugin>
         </sensor>
-    </link>
+        <material>Gazebo/Yellow</material>
+    </gazebo>
     <joint name="base_to_imu" type="fixed">
+        <origin xyz="0 0 ${wheel_diameter}" rpy="0 0 0"/>
         <parent link="base_link"/>
         <child link="imu_link"/>
@@ -29,5 +42,5 @@
     <link name="sllidar_base_link">
         <visual>
-            <origin xyz="${wheelbase_length / 2} 0 ${wheel_diameter * 1.5}" rpy="0 0 0"/>
+            <origin xyz="0 0 0" rpy="0 0 0"/>
             <geometry>
                 <cylinder length="${lidar_size}" radius="${lidar_size}"/>
@@ -35,41 +48,47 @@
             <material name="lidar_material"/>
         </visual>
-        <sensor name="lidar" type="gpu_ray">
+        <collision>
+            <origin xyz="0 0 0" rpy="0 0 0"/>
+            <geometry>
+                <cylinder length="${lidar_size}" radius="${lidar_size}"/>
+            </geometry>
+        </collision>
+        <inertial>
+            <mass value="0.2"/>
+            <origin xyz="0 0 0" rpy="0 0 0"/>
+            <inertia ixx="0.0001" ixy="0.0" ixz="0.0" iyy="0.0001" iyz="0.0" izz="0.0001"/>
+        </inertial>
+    </link>
+    <gazebo reference="sllidar_base_link">
+        <sensor name="sensor_gpu_ray" type="ray">
+            <visualize>false</visualize>
             <ray>
                 <scan>
                     <horizontal>
-                        <samples>720</samples>
-                        <resolution>1</resolution>
-                        <min_angle>-${pi / 2}</min_angle>
-                        <max_angle>${pi / 2}</max_angle>
+                        <samples>360</samples>
+                        <resolution>1.0</resolution>
+                        <min_angle>-${pi}</min_angle>
+                        <max_angle>${pi}</max_angle>
                     </horizontal>
                 </scan>
                 <range>
-                    <min>0.10</min>
-                    <max>30.0</max>
-                    <resolution>0.01</resolution>
+                    <min>0.5</min>
+                    <max>50.0</max>
                 </range>
-              <!-- Using gazebo's noise instead of plugin's -->
-                <noise>
-                    <type>gaussian</type>
-                    <mean>0.0</mean>
-                    <stddev>0.01</stddev>
-                </noise>
             </ray>
-            <!-- Using gazebo's update rate instead of plugin's -->
-            <update_rate>30</update_rate>
-            <plugin name="my_lidar" filename="libgazebo_ros_ray_sensor.so">
-                <!-- Change namespace and output topic so published topic is /rrbot/laser/scan -->
-                <ros>
-                    <namespace>/rrbot/laser</namespace>
-                    <remapping>~/out:=scan</remapping>
-                </ros>
-              <!-- Set output to sensor_msgs/LaserScan to get same output type as gazebo_ros_laser -->
+            <always_on>true</always_on>
+            <plugin name="laser_scan_plugin" filename="libgazebo_ros_ray_sensor.so">
                 <output_type>sensor_msgs/LaserScan</output_type>
-              <!-- <frame_name> ommited, will default to hokuo_link -->
+                <frameName>sllidar_base_link</frameName>
+                <topicName>/scan</topicName>
+                <remapping>~/out:=scan</remapping>
+                <robotNamespace>/</robotNamespace>
+                <updateRate>30.0</updateRate>
             </plugin>
         </sensor>
-    </link>
+        <material>Gazebo/Purple</material>
+    </gazebo>
     <joint name="base_to_lidar" type="fixed">
+        <origin xyz="${wheelbase_length / 2} 0 ${wheel_diameter * 1.5}" rpy="0 0 0"/>
         <parent link="base_link"/>
         <child link="sllidar_base_link"/>

File: smartcar_simulation/urdf/smartcar.urdf.xacro (robot description, xacro)
@@ -10,4 +10,5 @@
     </link>
     <joint name="base_to_chassis" type="fixed">
+        <origin xyz="0 0 ${wheel_radius}" rpy="0 0 0"/>
         <parent link="base_link"/>
         <child link="chassis_link"/>
@@ -18,24 +19,45 @@
                 <box size="${wheelbase_length} ${wheelbase_width} ${chassis_thickness}"/>
             </geometry>
-            <origin xyz="0 0 ${wheel_radius}" rpy="0 0 0"/>
+            <origin xyz="0 0 0" rpy="0 0 0"/>
+            <material name="body_material"/>
         </visual>
+        <collision>
+            <geometry>
+                <box size="${wheelbase_length} ${wheelbase_width} ${chassis_thickness}"/>
+            </geometry>
+            <origin xyz="0 0 0" rpy="0 0 0"/>
+        </collision>
+        <inertial>
+            <mass value="5.0"/>
+            <origin xyz="0 0 0" rpy="0 0 0"/>
+            <inertia ixx="0.02" ixy="0.0" ixz="0.0" iyy="0.02" iyz="0.0" izz="0.02"/>
+        </inertial>
     </link>
-    <link name="base_footprint">
-        <visual>
-            <geometry>
-                <box size="${wheelbase_length * 2} ${wheelbase_width * 2} ${wheel_diameter * 2}"/>
-            </geometry>
-            <material name="footprint_material"/>
-            <origin xyz="0 0 ${wheel_diameter}" rpy="0 0 0" />
-        </visual>
-    </link>
+    <gazebo reference="chassis_link">
+        <material>Gazebo/Red</material>
+    </gazebo>
     <joint name="base_to_footprint" type="fixed">
         <parent link="base_link"/>
         <child link="base_footprint"/>
     </joint>
+    <link name="base_footprint">
+        <visual>
+            <origin xyz="0 0 0.0001" rpy="0 0 0" />
+            <geometry>
+                <box size="${wheelbase_length} ${wheelbase_width} 0"/>
+            </geometry>
+            <material name="footprint_material"/>
+        </visual>
+    </link>
+    <gazebo reference="base_footprint">
+        <material>Gazebo/TurquoiseGlow</material>
+    </gazebo>
     <xacro:front_wheel prefix="left" parent="base_link" x="${wheelbase_length / 2}" y="${wheelbase_width / 2}" z="${wheel_radius}" wheel_offset="${wheel_width / 2}"/>
     <xacro:front_wheel prefix="right" parent="base_link" x="${wheelbase_length / 2}" y="-${wheelbase_width / 2}" z="${wheel_radius}" wheel_offset="-${wheel_width / 2}"/>
-    <xacro:rear_wheel prefix="left" parent="base_link" x="-${wheelbase_length / 2}" y="${wheelbase_width / 2}" z="${wheel_radius}" wheel_offset="${wheel_width / 2}"/>
-    <xacro:rear_wheel prefix="right" parent="base_link" x="-${wheelbase_length / 2}" y="-${wheelbase_width / 2}" z="${wheel_radius}" wheel_offset="-${wheel_width / 2}"/>
+    <xacro:back_wheel prefix="left" parent="base_link" x="-${wheelbase_length / 2}" y="${wheelbase_width / 2}" z="${wheel_radius}" wheel_offset="${wheel_width / 2}"/>
+    <xacro:back_wheel prefix="right" parent="base_link" x="-${wheelbase_length / 2}" y="-${wheelbase_width / 2}" z="${wheel_radius}" wheel_offset="-${wheel_width / 2}"/>
     <xacro:include filename="sensors.xacro"/>
+    <gazebo>
+        <plugin name="car_gazebo_plugin" filename="libcar_gazebo_plugin.so"></plugin>
+    </gazebo>
 </robot>

File: smartcar_simulation/urdf/wheels.xacro (robot description, xacro)
@@ -5,4 +5,5 @@
     <xacro:property name="wheel_width" value="0.025"/>
     <xacro:property name="wheel_oriantation" value="${90 * (pi / 180)}"/>
+    <xacro:property name="steer_link_size" value="0.01"/>
     <xacro:macro name="front_wheel" params="prefix parent x y z wheel_offset">
         <joint name="front_${prefix}_wheel_steer_joint" type="revolute">
@@ -15,5 +16,25 @@
         <link name="front_${prefix}_wheel_steer_link">
             <origin xyz="0 0 0" rpy="0 0 0" />
+            <visual>
+                <geometry>
+                    <box size="${steer_link_size} ${steer_link_size} ${steer_link_size}"/>
+                </geometry>
+                <origin xyz="0 0 0" rpy="0 0 0"/>
+            </visual>
+            <collision>
+                <geometry>
+                    <box size="${steer_link_size} ${steer_link_size} ${steer_link_size}"/>
+                </geometry>
+                <origin xyz="0 0 0" rpy="0 0 0"/>
+            </collision>
+            <inertial>
+                <mass value="0.1"/>
+                <origin xyz="0 0 0" rpy="0 0 0"/>
+                <inertia ixx="0.00005" ixy="0.0" ixz="0.0" iyy="0.00005" iyz="0.0" izz="0.00005"/>
+            </inertial>
         </link>
+        <gazebo reference="front_${prefix}_wheel_steer_link">
+            <material>Gazebo/Red</material>
+        </gazebo>
         <joint name="front_${prefix}_wheel_joint" type="continuous">
             <origin xyz="0 0 0" rpy="0 0 0" />
@@ -30,22 +51,50 @@
                 <material name="wheel_material"/>
             </visual>
+            <collision>
+                <geometry>
+                    <cylinder length="${wheel_width}" radius="${wheel_radius}"/>
+                </geometry>
+                <origin xyz="0 ${wheel_offset} 0" rpy="${wheel_oriantation} 0 0"/>
+            </collision>
+            <inertial>
+                <mass value="0.2"/>
+                <origin xyz="0 0 0" rpy="0 0 0"/>
+                <inertia ixx="0.0001" ixy="0.0" ixz="0.0" iyy="0.0001" iyz="0.0" izz="0.0001"/>
+            </inertial>
         </link>
+        <gazebo reference="front_${prefix}_wheel_link">
+            <material>Gazebo/Black</material>
+        </gazebo>
     </xacro:macro>
-    <xacro:macro name="rear_wheel" params="prefix parent x y z wheel_offset">
-        <joint name="rear_${prefix}_wheel_joint" type="continuous">
+    <xacro:macro name="back_wheel" params="prefix parent x y z wheel_offset">
+        <joint name="back_${prefix}_wheel_joint" type="continuous">
             <origin xyz="${x} ${y} ${z}" rpy="0 0 0"/>
             <parent link="${parent}"/>
-            <child link="rear_${prefix}_wheel_link"/>
+            <child link="back_${prefix}_wheel_link"/>
             <axis xyz="0 1 0"/>
         </joint>
-        <link name="rear_${prefix}_wheel_link">
+        <link name="back_${prefix}_wheel_link">
             <visual>
                 <geometry>
                     <cylinder length="${wheel_width}" radius="${wheel_radius}"/>
                 </geometry>
-                <origin xyz="0 ${wheel_offset} 0" rpy="${wheel_oriantation} 0 0" />
+                <origin xyz="0 ${wheel_offset} 0" rpy="${wheel_oriantation} 0 0"/>
                 <material name="wheel_material"/>
             </visual>
+            <collision>
+                <geometry>
+                    <cylinder length="${wheel_width}" radius="${wheel_radius}"/>
+                </geometry>
+                <origin xyz="0 ${wheel_offset} 0" rpy="${wheel_oriantation} 0 0"/>
+            </collision>
+            <inertial>
+                <mass value="0.2"/>
+                <origin xyz="0 0 0" rpy="0 0 0"/>
+                <inertia ixx="0.0001" ixy="0.0" ixz="0.0" iyy="0.0001" iyz="0.0" izz="0.0001"/>
+            </inertial>
         </link>
+        <gazebo reference="back_${prefix}_wheel_link">
+            <material>Gazebo/Black</material>
+        </gazebo>
     </xacro:macro>
 </robot>

Commit message: removed old files

File: smartcar_simulation/urdf/materials.xacro (robot description, xacro)
@@ -11,5 +11,5 @@
     </material>
     <material name="lidar_material">
-        <color rgba="1 0 1 1"/>
+        <color rgba="0 0 0 1"/>
     </material>
     <material name="footprint_material">

File: smartcar_simulation/urdf/sensors.xacro (robot description, xacro)
@@ -73,5 +73,5 @@
                 </scan>
                 <range>
-                    <min>0.5</min>
+                    <min>0.3</min>
                     <max>50.0</max>
                 </range>
@@ -83,9 +83,8 @@
                 <topicName>/scan</topicName>
                 <remapping>~/out:=scan</remapping>
-                <robotNamespace>/</robotNamespace>
                 <updateRate>30.0</updateRate>
             </plugin>
         </sensor>
-        <material>Gazebo/Purple</material>
+        <material>Gazebo/Black</material>
     </gazebo>
     <joint name="base_to_lidar" type="fixed">
